Commit message: kumi_bringup working and traj_control also

File: src/kumi_description/urdf/core.xacro (robot description, xacro)
@@ -1,10 +1,4 @@
 <?xml version="1.0" ?>
 <robot xmlns:xacro="http://www.ros.org/wiki/xacro" name="kumi">
-    <xacro:property name="mesh_scale" value="0.001 0.001 0.001"/>
-    <xacro:property name="mesh_dir" value="file://${kumi_share}/meshes"/>
-    <xacro:property name="body_mesh" value="${mesh_dir}/body_v5.STL"/>
-    <xacro:property name="leg_mesh" value="${mesh_dir}/leg_v2.stl"/>
-    <xacro:property name="foot_mesh" value="${mesh_dir}/piedino_v3.STL"/>
-    <xacro:property name="realsense_mesh" value="${mesh_dir}/realsense.stl"/>
     <link name="body">
         <visual>
@@ -13,7 +7,5 @@
                 <mesh filename="${body_mesh}" scale="${mesh_scale}"/>
             </geometry>
-            <material name="gray">
-                <color rgba="0 0 0 0.8"/>
-            </material>
+            <material name="gray"/>
         </visual>
         <collision>
@@ -37,14 +29,4 @@
         <dynamics damping="0.5" friction="${joint_friction}"/>
     </joint>
-    <gazebo reference="front_sh">
-        <sensor name="front_sh_force_torque" type="force_torque">
-            <always_on>true</always_on>
-            <update_rate>500</update_rate>
-            <force_torque>
-                <frame>child</frame>
-                <measure_direction>child_to_parent</measure_direction>
-            </force_torque>
-        </sensor>
-    </gazebo>
     <link name="front_leg">
         <visual>
@@ -53,7 +35,5 @@
                 <mesh filename="${leg_mesh}" scale="${mesh_scale}"/>
             </geometry>
-            <material name="gray">
-                <color rgba="0 0 0 0.8"/>
-            </material>
+            <material name="gray"/>
         </visual>
         <collision>
@@ -76,73 +56,22 @@
     <link name="realsense">
         <visual>
-            <origin xyz="-0.025 0 -0.057" rpy="${pi/2} 0  ${-pi/2}"/>
+            <origin xyz="-0.025 0 -0.057" rpy="${pi/2} 0 0"/>
             <geometry>
-                <mesh filename="${realsense_mesh}" scale="${mesh_scale}"/>
+                <box size="0.03 0.03 0.06"/>
             </geometry>
-            <material name="green">
-                <color rgba="0 1 0 1"/>
-            </material>
+            <material name="green"/>
         </visual>
         <collision>
-            <origin xyz="-0.025 0 -0.057" rpy="${pi/2} 0  ${-pi/2}"/>
+            <origin xyz="-0.025 0 -0.057" rpy="${pi/2} 0 0"/>
             <geometry>
-                <mesh filename="${realsense_mesh}" scale="${mesh_scale}"/>
+                <box size="0.03 0.03 0.06"/>
             </geometry>
         </collision>
         <inertial>
-            <origin xyz="-0.025 0 -0.057" rpy="${pi/2} 0  ${-pi/2}"/>
+            <origin xyz="-0.025 0 -0.057" rpy="${pi/2} 0 0"/>
             <mass value="0.005"/>
             <inertia ixx="0.000091" ixy="0.0" ixz="0.0" iyy="0.000165" iyz="0.0" izz="0.000091"/>
         </inertial>
     </link>
-    <gazebo reference="realsense">
-        <sensor name="realsense" type="rgbd_camera">
-            <pose>-0.025 0 -0.057 0 0 3.14159</pose>
-            <always_on>1</always_on>
-            <update_rate>100</update_rate>
-            <topic>/d435_rgbd</topic>
-            <frameName>realsense</frameName>
-            <camera name="rs_front">
-                <horizontal_fov>1.50098</horizontal_fov>
-                <lens>
-                    <intrinsics>
-                    <fx>343.159</fx>
-                    <fy>343.159</fy>
-                    <cx>319.5</cx>
-                    <cy>179.5</cy>
-                    <s>0</s>
-                    </intrinsics>
-                </lens>
-                <distortion>
-                    <k1>0.0</k1>
-                    <k2>0.0</k2>
-                    <k3>0.0</k3>
-                    <p1>0.0</p1>
-                    <p2>0.0</p2>
-                    <center>0.5 0.5</center>
-                </distortion>
-                <image>
-                    <width>640</width>
-                    <height>360</height>
-                    <format>R8G8B8</format>
-                </image>
-                <clip>
-                    <near>0.01</near>
-                    <far>300</far>
-                </clip>
-                <depth_camera>
-                    <clip>
-                    <near>0.1</near>
-                    <far>10</far>
-                    </clip>
-                </depth_camera>
-                <noise>
-                    <type>gaussian</type>
-                    <mean>0</mean>
-                    <stddev>0.007</stddev>
-                </noise>
-            </camera>
-        </sensor>
-    </gazebo>
     <joint name="front_ank_y" type="revolute">
         <origin xyz="0 0 ${-leg_len}" rpy="0 0 0"/>
@@ -153,14 +82,4 @@
         <dynamics damping="0.1" friction="${joint_friction}"/>
     </joint>
-    <gazebo reference="front_ank_y">
-        <sensor name="front_ank_force_torque" type="force_torque">
-            <always_on>true</always_on>
-            <update_rate>500</update_rate>
-            <force_torque>
-                <frame>child</frame>
-                <measure_direction>child_to_parent</measure_direction>
-            </force_torque>
-        </sensor>
-    </gazebo>
     <link name="front_foot_dummy">
         <inertial>
@@ -178,26 +97,14 @@
         <dynamics damping="0.1" friction="${joint_friction}"/>
     </joint>
-    <gazebo reference="front_ank_z">
-        <sensor name="front_ank_force_torque" type="force_torque">
-            <always_on>true</always_on>
-            <update_rate>500</update_rate>
-            <force_torque>
-                <frame>child</frame>
-                <measure_direction>child_to_parent</measure_direction>
-            </force_torque>
-        </sensor>
-    </gazebo>
     <link name="front_foot">
         <visual>
-            <origin xyz="0 -0.007 0" rpy="${pi/2} 0  ${-pi/2}"/>
+            <origin xyz="0 -0.007 0" rpy="${pi/2} 0 ${-pi/2}"/>
             <geometry>
                 <mesh filename="${foot_mesh}" scale="${mesh_scale}"/>
             </geometry>
-            <material name="green">
-                <color rgba="0 1 0 0.8"/>
-            </material>
+            <material name="green"/>
         </visual>
         <collision name="frontFootCollision">
-            <origin xyz="0 0 0" rpy="${pi/2} 0  ${-pi/2}"/>
+            <origin xyz="0 0 0" rpy="${pi/2} 0 ${-pi/2}"/>
             <geometry>
                 <mesh filename="${foot_mesh}" scale="${mesh_scale}"/>
@@ -205,5 +112,5 @@
         </collision>
         <inertial>
-            <origin xyz="0 0 0" rpy="${pi/2} 0  ${-pi/2}"/>
+            <origin xyz="0 0 0" rpy="${pi/2} 0 ${-pi/2}"/>
             <mass value="0.15"/>
             <inertia ixx="0.000091" ixy="0.0" ixz="0.0" iyy="0.000165" iyz="0.0" izz="0.000091"/>
@@ -218,14 +125,4 @@
         <dynamics damping="0.5" friction="${joint_friction}"/>
     </joint>
-    <gazebo reference="rear_sh">
-        <sensor name="rear_sh_force_torque" type="force_torque">
-            <always_on>true</always_on>
-            <update_rate>500</update_rate>
-            <force_torque>
-                <frame>child</frame>
-                <measure_direction>child_to_parent</measure_direction>
-            </force_torque>
-        </sensor>
-    </gazebo>
     <link name="rear_leg">
         <visual>
@@ -234,7 +131,5 @@
                 <mesh filename="${leg_mesh}" scale="${mesh_scale}"/>
             </geometry>
-            <material name="gray">
-                <color rgba="0 0 0 0.8"/>
-            </material>
+            <material name="gray"/>
         </visual>
         <collision>
@@ -258,14 +153,4 @@
         <dynamics damping="0.1" friction="${joint_friction}"/>
     </joint>
-    <gazebo reference="rear_ank_y">
-        <sensor name="rear_ank_force_torque" type="force_torque">
-            <always_on>true</always_on>
-            <update_rate>500</update_rate>
-            <force_torque>
-                <frame>child</frame>
-                <measure_direction>child_to_parent</measure_direction>
-            </force_torque>
-        </sensor>
-    </gazebo>
     <link name="rear_foot_dummy">
         <inertial>
@@ -283,26 +168,14 @@
         <dynamics damping="0.1" friction="${joint_friction}"/>
     </joint>
-    <gazebo reference="rear_ank_z">
-        <sensor name="front_ank_force_torque" type="force_torque">
-            <always_on>true</always_on>
-            <update_rate>500</update_rate>
-            <force_torque>
-                <frame>child</frame>
-                <measure_direction>child_to_parent</measure_direction>
-            </force_torque>
-        </sensor>
-    </gazebo>
     <link name="rear_foot">
         <visual>
-            <origin xyz="0 0.007 0" rpy="${pi/2} 0  ${pi/2}"/>
+            <origin xyz="0 0.007 0" rpy="${pi/2} 0 ${pi/2}"/>
             <geometry>
                 <mesh filename="${foot_mesh}" scale="${mesh_scale}"/>
             </geometry>
-            <material name="red">
-                <color rgba="1 0 0 0.8"/>
-            </material>
+            <material name="red"/>
         </visual>
         <collision name="rearFootCollision">
-            <origin xyz="0 0 0" rpy="${pi/2} 0  ${pi/2}"/>
+            <origin xyz="0 0 0" rpy="${pi/2} 0 ${pi/2}"/>
             <geometry>
                 <mesh filename="${foot_mesh}" scale="${mesh_scale}"/>
@@ -310,5 +183,5 @@
         </collision>
         <inertial>
-            <origin xyz="0 0 0" rpy="${pi/2} 0  ${pi/2}"/>
+            <origin xyz="0 0 0" rpy="${pi/2} 0 ${pi/2}"/>
             <mass value="0.15"/>
             <inertia ixx="0.000091" ixy="0.0" ixz="0.0" iyy="0.000165" iyz="0.0" izz="0.000091"/>

File: src/kumi_description/urdf/kumi.xacro (robot description, xacro)
@@ -1,8 +1,9 @@
 <?xml version="1.0" ?>
 <robot xmlns:xacro="http://www.ros.org/wiki/xacro"  name="kumi">
-    <xacro:property name="kumi_share" value="$(find kumi_description)"/>
-    <xacro:include filename="${kumi_share}/urdf/variables.xacro" />
-    <xacro:include filename="${kumi_share}/urdf/trajectory_control.xacro" />
-    <xacro:include filename="${kumi_share}/urdf/kumi_mesh_stereocamera.xacro" />
-    <xacro:include filename="${kumi_share}/urdf/sensors_config.xacro" />
+    <xacro:arg name="pkg_share" default="$(find kumi_description)" />
+    <xacro:property name="pkg_share" value="$(arg pkg_share)"/>
+    <xacro:include filename="${pkg_share}/urdf/macros.xacro" />
+    <xacro:include filename="${pkg_share}/urdf/core.xacro" />
+    <xacro:include filename="${pkg_share}/urdf/sensors.xacro" />
+    <xacro:include filename="${pkg_share}/urdf/gazebo_plugins.xacro" />
 </robot>

Commit message: new gz gui with robot control, started to create a structure that allowes multiple robots spawn with separate controllers

File: src/kumi_description/urdf/core.xacro (robot description, xacro)
@@ -117,4 +117,8 @@
         </inertial>
     </link>
+    <gazebo reference="front_foot">
+        <mu1>${foot_contact_friction}</mu1>
+        <mu2>${foot_contact_friction}</mu2>
+    </gazebo>
     <joint name="rear_sh" type="revolute">
         <origin xyz="${lenght/2} 0.006 0" rpy="0 0 0"/>
@@ -188,3 +192,7 @@
         </inertial>
     </link>
+    <gazebo reference="rear_foot">
+        <mu1>${foot_contact_friction}</mu1>
+        <mu2>${foot_contact_friction}</mu2>
+    </gazebo>
 </robot>

File: src/kumi_description/urdf/kumiiiii.xacro (robot description, xacro)
@@ -61,6 +61,6 @@
     <inertial>
       <origin rpy="0 -1.5707963267948966 0" xyz="0 0 0"/>
-      <mass value="0.3"/>
-      <inertia ixx="0.000023773" ixy="0.0" ixz="0.0" iyy="0.000513246" iyz="0.0" izz="0.000524232"/>
+      <mass value="0.212"/>
+      <inertia ixx="0.001148663" ixy="0.0" ixz="0.0" iyy="0.001120663" iyz="-0.000045" izz="0.000046"/>
     </inertial>
   </link>
@@ -133,4 +133,8 @@
     </inertial>
   </link>
+  <gazebo reference="front_foot">
+    <mu1>2.0</mu1>
+    <mu2>2.0</mu2>
+  </gazebo>
   <joint name="rear_sh" type="revolute">
     <origin rpy="0 0 0" xyz="0.09 0.006 0"/>
@@ -157,6 +161,6 @@
     <inertial>
       <origin rpy="0 -1.5707963267948966 3.141592653589793" xyz="0 0 0"/>
-      <mass value="0.3"/>
-      <inertia ixx="0.000023773" ixy="0.0" ixz="0.0" iyy="0.000513246" iyz="0.0" izz="0.000524232"/>
+      <mass value="0.212"/>
+      <inertia ixx="0.001148663" ixy="0.0" ixz="0.0" iyy="0.001120663" iyz="-0.000045" izz="0.000046"/>
     </inertial>
   </link>
@@ -204,4 +208,8 @@
     </inertial>
   </link>
+  <gazebo reference="rear_foot">
+    <mu1>2.0</mu1>
+    <mu2>2.0</mu2>
+  </gazebo>
   <link name="front_camera">
     <visual>

File: src/kumi_description/urdf/macros.xacro (robot description, xacro)
@@ -18,4 +18,5 @@
     <xacro:property name="mass" value="0.3" />
     <xacro:property name="joint_friction" value="0.2" />
+    <xacro:property name="foot_contact_friction" value="2.0" />
     <xacro:property name="mesh_scale" value="0.001 0.001 0.001"/>
     <xacro:property name="body_mesh" value="${mesh_dir}/body_v5.STL"/>

File: src/kumi_description/urdf/sensors.xacro (robot description, xacro)
@@ -25,5 +25,5 @@
             <parent link="realsense"/>
             <child link="front_camera"/>
-            <origin xyz="0 0 0" rpy="0 0 0"/>
+            <origin xyz="-0.03 0 0" rpy="0 0 3.141592653589793"/>
         </joint>
         <gazebo reference="front_camera">
@@ -32,6 +32,6 @@
                 <visualize>true</visualize>
                 <update_rate>30</update_rate>
-                <topic>front_camera/image</topic>
-                <camera_info_topic>front_camera/camera_info</camera_info_topic>
+                <topic>$(arg ros_namespace)/front_camera/image</topic>
+                <camera_info_topic>$(arg ros_namespace)/front_camera/camera_info</camera_info_topic>
                 <gz_frame_id>front_camera</gz_frame_id>
                 <camera>
@@ -72,5 +72,5 @@
             <parent link="realsense"/>
             <child link="front_depth"/>
-            <origin xyz="0.005 0 0" rpy="0 0 0"/>
+            <origin xyz="-0.035 0 0.015" rpy="0 0 3.141592653589793"/>
         </joint>
         <gazebo reference="front_depth">
@@ -79,6 +79,6 @@
                 <visualize>true</visualize>
                 <update_rate>20</update_rate>
-                <topic>front_depth/image</topic>
-                <camera_info_topic>front_depth/camera_info</camera_info_topic>
+                <topic>$(arg ros_namespace)/front_depth/image</topic>
+                <camera_info_topic>$(arg ros_namespace)/front_depth/camera_info</camera_info_topic>
                 <gz_frame_id>front_depth</gz_frame_id>
                 <camera>
