Commit message: working

File: src/kumi_description/urdf/kumiiiii.xacro (robot description, xacro)
@@ -1,7 +1,3 @@
 <?xml version="1.0" ?>
-<!-- =================================================================================== -->
-<!-- |    This document was autogenerated by xacro from /home/andreas/dev_ws/kumi_stack/src/kumi_description/urdf/kumi.xacro | -->
-<!-- |    EDITING THIS FILE BY HAND IS NOT RECOMMENDED                                 | -->
-<!-- =================================================================================== -->
 <robot name="kumi">
   <material name="black">
@@ -9,5 +5,5 @@
   </material>
   <material name="gray">
-    <color rgba="0 0 0 0.8"/>
+    <color rgba="0.5 0.5 0.5 0.8"/>
   </material>
   <material name="green">
@@ -17,9 +13,10 @@
     <color rgba="1 0 0 0.8"/>
   </material>
+  <!-- ========== BODY ========== -->
   <link name="body">
     <visual>
       <origin rpy="0 0 0" xyz="0 0 0"/>
       <geometry>
-        <mesh filename="/home/andreas/dev_ws/kumi_stack/install/kumi_description/share/kumi_description/meshes/body_v5.STL" scale="0.001 0.001 0.001"/>
+        <mesh filename="meshes/body_v5.STL" scale="0.001 0.001 0.001"/>
       </geometry>
       <material name="gray"/>
@@ -28,5 +25,5 @@
       <origin rpy="0 0 0" xyz="0 0 0"/>
       <geometry>
-        <mesh filename="/home/andreas/dev_ws/kumi_stack/install/kumi_description/share/kumi_description/meshes/body_v5.STL" scale="0.001 0.001 0.001"/>
+        <mesh filename="meshes/body_v5.STL" scale="0.001 0.001 0.001"/>
       </geometry>
     </collision>
@@ -37,4 +34,5 @@
     </inertial>
   </link>
+  <!-- ========== FRONT LEG ========== -->
   <joint name="front_sh" type="revolute">
     <origin rpy="0 0 0" xyz="-0.09 -0.006 0"/>
@@ -49,5 +47,5 @@
       <origin rpy="0 -1.5707963267948966 0" xyz="0 0 0"/>
       <geometry>
-        <mesh filename="/home/andreas/dev_ws/kumi_stack/install/kumi_description/share/kumi_description/meshes/leg_v2.stl" scale="0.001 0.001 0.001"/>
+        <mesh filename="meshes/leg_v2.stl" scale="0.001 0.001 0.001"/>
       </geometry>
       <material name="gray"/>
@@ -56,5 +54,5 @@
       <origin rpy="0 -1.5707963267948966 0" xyz="0 0 0"/>
       <geometry>
-        <mesh filename="/home/andreas/dev_ws/kumi_stack/install/kumi_description/share/kumi_description/meshes/leg_v2.stl" scale="0.001 0.001 0.001"/>
+        <mesh filename="meshes/leg_v2.stl" scale="0.001 0.001 0.001"/>
       </geometry>
     </collision>
@@ -65,29 +63,5 @@
     </inertial>
   </link>
-  <joint name="realsense_joint" type="fixed">
-    <origin rpy="0 0 0" xyz="0 0 0"/>
-    <parent link="front_leg"/>
-    <child link="realsense"/>
-  </joint>
-  <link name="realsense">
-    <visual>
-      <origin rpy="1.5707963267948966 0 -1.5707963267948966" xyz="-0.025 0 -0.057"/>
-      <geometry>
-        <box size="0.03 0.03 0.06"/>
-      </geometry>
-      <material name="green"/>
-    </visual>
-    <collision>
-      <origin rpy="1.5707963267948966 0 -1.5707963267948966" xyz="-0.025 0 -0.057"/>
-      <geometry>
-        <box size="0.03 0.03 0.06"/>
-      </geometry>
-    </collision>
-    <inertial>
-      <origin rpy="1.5707963267948966 0 -1.5707963267948966" xyz="-0.025 0 -0.057"/>
-      <mass value="0.005"/>
-      <inertia ixx="0.000091" ixy="0.0" ixz="0.0" iyy="0.000165" iyz="0.0" izz="0.000091"/>
-    </inertial>
-  </link>
+  <!-- ========== FRONT ANKLE ========== -->
   <joint name="front_ank_y" type="revolute">
     <origin rpy="0 0 0" xyz="0 0 -0.11"/>
@@ -117,12 +91,12 @@
       <origin rpy="1.5707963267948966 0 -1.5707963267948966" xyz="0 -0.007 0"/>
       <geometry>
-        <mesh filename="/home/andreas/dev_ws/kumi_stack/install/kumi_description/share/kumi_description/meshes/piedino_v3.STL" scale="0.001 0.001 0.001"/>
+        <mesh filename="meshes/piedino_v3.STL" scale="0.001 0.001 0.001"/>
       </geometry>
       <material name="green"/>
     </visual>
-    <collision name="frontFootCollision">
+    <collision>
       <origin rpy="1.5707963267948966 0 -1.5707963267948966" xyz="0 0 0"/>
       <geometry>
-        <mesh filename="/home/andreas/dev_ws/kumi_stack/install/kumi_description/share/kumi_description/meshes/piedino_v3.STL" scale="0.001 0.001 0.001"/>
+        <mesh filename="meshes/piedino_v3.STL" scale="0.001 0.001 0.001"/>
       </geometry>
     </collision>
@@ -133,8 +107,5 @@
     </inertial>
   </link>
-  <gazebo reference="front_foot">
-    <mu1>2.0</mu1>
-    <mu2>2.0</mu2>
-  </gazebo>
+  <!-- ========== REAR LEG ========== -->
   <joint name="rear_sh" type="revolute">
     <origin rpy="0 0 0" xyz="0.09 0.006 0"/>
@@ -149,5 +120,5 @@
       <origin rpy="0 -1.5707963267948966 3.141592653589793" xyz="0 0 0"/>
       <geometry>
-        <mesh filename="/home/andreas/dev_ws/kumi_stack/install/kumi_description/share/kumi_description/meshes/leg_v2.stl" scale="0.001 0.001 0.001"/>
+        <mesh filename="meshes/leg_v2.stl" scale="0.001 0.001 0.001"/>
       </geometry>
       <material name="gray"/>
@@ -156,5 +127,5 @@
       <origin rpy="0 -1.5707963267948966 3.141592653589793" xyz="0 0 0"/>
       <geometry>
-        <mesh filename="/home/andreas/dev_ws/kumi_stack/install/kumi_description/share/kumi_description/meshes/leg_v2.stl" scale="0.001 0.001 0.001"/>
+        <mesh filename="meshes/leg_v2.stl" scale="0.001 0.001 0.001"/>
       </geometry>
     </collision>
@@ -165,4 +136,5 @@
     </inertial>
   </link>
+  <!-- ========== REAR ANKLE ========== -->
   <joint name="rear_ank_y" type="revolute">
     <origin rpy="0 0 0" xyz="0 0 -0.11"/>
@@ -192,12 +164,12 @@
       <origin rpy="1.5707963267948966 0 1.5707963267948966" xyz="0 0.007 0"/>
       <geometry>
-        <mesh filename="/home/andreas/dev_ws/kumi_stack/install/kumi_description/share/kumi_description/meshes/piedino_v3.STL" scale="0.001 0.001 0.001"/>
+        <mesh filename="meshes/piedino_v3.STL" scale="0.001 0.001 0.001"/>
       </geometry>
       <material name="red"/>
     </visual>
-    <collision name="rearFootCollision">
+    <collision>
       <origin rpy="1.5707963267948966 0 1.5707963267948966" xyz="0 0 0"/>
       <geometry>
-        <mesh filename="/home/andreas/dev_ws/kumi_stack/install/kumi_description/share/kumi_description/meshes/piedino_v3.STL" scale="0.001 0.001 0.001"/>
+        <mesh filename="meshes/piedino_v3.STL" scale="0.001 0.001 0.001"/>
       </geometry>
     </collision>
@@ -208,101 +180,29 @@
     </inertial>
   </link>
-  <gazebo reference="rear_foot">
-    <mu1>2.0</mu1>
-    <mu2>2.0</mu2>
-  </gazebo>
-  <link name="front_camera">
-    <visual>
-      <origin rpy="0 0 0" xyz="0 0 0"/>
-      <geometry>
-        <box size="0.01 0.01 0.01"/>
-      </geometry>
-      <material name="black"/>
-    </visual>
-    <collision>
-      <origin rpy="0 0 0" xyz="0 0 0"/>
-      <geometry>
-        <box size="0.01 0.01 0.01"/>
-      </geometry>
-    </collision>
-    <inertial>
-      <origin rpy="0 0 0" xyz="0 0 0"/>
-      <mass value="0.01"/>
-      <inertia ixx="1e-6" ixy="0" ixz="0" iyy="1e-6" iyz="0" izz="1e-6"/>
-    </inertial>
-  </link>
-  <joint name="front_camera_joint" type="fixed">
-    <parent link="realsense"/>
-    <child link="front_camera"/>
+  <!-- ========== REALSENSE (struttura, no sensori) ========== -->
+  <joint name="realsense_joint" type="fixed">
     <origin rpy="0 0 0" xyz="0 0 0"/>
-  </joint>
-  <gazebo reference="front_camera">
-    <sensor name="front_camera" type="camera">
-      <always_on>true</always_on>
-      <visualize>true</visualize>
-      <update_rate>30</update_rate>
-      <topic>front_camera/image</topic>
-      <camera_info_topic>front_camera/camera_info</camera_info_topic>
-      <gz_frame_id>front_camera</gz_frame_id>
-      <camera>
-        <horizontal_fov>1.3962634</horizontal_fov>
-        <image>
-          <width>1280</width>
-          <height>720</height>
-          <format>R8G8B8</format>
-        </image>
-        <clip>
-          <near>0.05</near>
-          <far>50.0</far>
-        </clip>
-      </camera>
-    </sensor>
-  </gazebo>
-  <link name="front_depth">
-    <visual>
-      <origin rpy="0 0 0" xyz="0 0 0"/>
-      <geometry>
-        <box size="0.012 0.012 0.012"/>
+    <parent link="front_leg"/>
+    <child link="realsense"/>
+  </joint>
+  <link name="realsense">
+    <visual>
+      <origin rpy="1.5707963267948966 0 -1.5707963267948966" xyz="-0.025 0 -0.057"/>
+      <geometry>
+        <box size="0.03 0.03 0.06"/>
       </geometry>
       <material name="green"/>
     </visual>
     <collision>
-      <origin rpy="0 0 0" xyz="0 0 0"/>
-      <geometry>
-        <box size="0.012 0.012 0.012"/>
-      </geometry>
-    </collision>
-    <inertial>
-      <origin rpy="0 0 0" xyz="0 0 0"/>
-      <mass value="0.015"/>
-      <inertia ixx="2e-6" ixy="0" ixz="0" iyy="2e-6" iyz="0" izz="2e-6"/>
-    </inertial>
-  </link>
-  <joint name="front_depth_joint" type="fixed">
-    <parent link="realsense"/>
-    <child link="front_depth"/>
-    <origin rpy="0 0 0" xyz="0.005 0 0"/>
-  </joint>
-  <gazebo reference="front_depth">
-    <sensor name="front_depth_camera" type="depth_camera">
-      <always_on>true</always_on>
-      <visualize>true</visualize>
-      <update_rate>20</update_rate>
-      <topic>front_depth/image</topic>
-      <camera_info_topic>front_depth/camera_info</camera_info_topic>
-      <gz_frame_id>front_depth</gz_frame_id>
-      <camera>
-        <horizontal_fov>1.22173</horizontal_fov>
-        <image>
-          <width>640</width>
-          <height>480</height>
-          <format>R_FLOAT32</format>
-        </image>
-        <clip>
-          <near>0.10</near>
-          <far>10.0</far>
-        </clip>
-      </camera>
-    </sensor>
-  </gazebo>
+      <origin rpy="1.5707963267948966 0 -1.5707963267948966" xyz="-0.025 0 -0.057"/>
+      <geometry>
+        <box size="0.03 0.03 0.06"/>
+      </geometry>
+    </collision>
+    <inertial>
+      <origin rpy="1.5707963267948966 0 -1.5707963267948966" xyz="-0.025 0 -0.057"/>
+      <mass value="0.005"/>
+      <inertia ixx="0.000091" ixy="0.0" ixz="0.0" iyy="0.000165" iyz="0.0" izz="0.000091"/>
+    </inertial>
+  </link>
 </robot>
