Commit message: manual walk, some bugsss

File: src/kumi_description/urdf/macros.xacro (robot description, xacro)
@@ -1,3 +1,3 @@
-<?xml version="1.0" ?>
+<?xml version="1.0"?>
 <robot xmlns:xacro="http://www.ros.org/wiki/xacro" name="kumi">
     <xacro:arg name="pkg_share" default="$(find kumi_description)" />
@@ -6,7 +6,8 @@
     <xacro:arg name="enable_sensors" default="true" />
     <xacro:arg name="use_sim" default="false" />
-    <xacro:arg name="control_config" default="$(find kumi_control)/config/trajectory_control_config.yaml" />
-    <xacro:property name="pkg_share" value="$(arg pkg_share)"/>
-    <xacro:property name="mesh_dir" value="${pkg_share}/meshes"/>
+    <xacro:arg name="control_config"
+        default="$(find kumi_control)/config/trajectory_control_config.yaml" />
+    <xacro:property name="pkg_share" value="$(arg pkg_share)" />
+    <xacro:property name="mesh_dir" value="${pkg_share}/meshes" />
     <xacro:property name="ang_low_lim" value="0.85" />
     <xacro:property name="ang_up_lim" value="4" />
@@ -19,12 +20,20 @@
     <xacro:property name="joint_friction" value="0.2" />
     <xacro:property name="foot_contact_friction" value="2.0" />
-    <xacro:property name="mesh_scale" value="0.001 0.001 0.001"/>
-    <xacro:property name="body_mesh" value="${mesh_dir}/body_v5.STL"/>
-    <xacro:property name="leg_mesh" value="${mesh_dir}/leg_v2.stl"/>
-    <xacro:property name="foot_mesh" value="${mesh_dir}/piedino_v3.STL"/>
-    <xacro:property name="realsense_mesh" value="${mesh_dir}/realsense.stl"/>
-    <material name="black"><color rgba="0.1 0.1 0.1 1.0"/></material>
-    <material name="gray"><color rgba="0 0 0 0.8"/></material>
-    <material name="green"><color rgba="0 1 0 0.8"/></material>
-    <material name="red"><color rgba="1 0 0 0.8"/></material>
+    <xacro:property name="mesh_scale" value="0.001 0.001 0.001" />
+    <xacro:property name="body_mesh" value="${mesh_dir}/body_v5.STL" />
+    <xacro:property name="leg_mesh" value="${mesh_dir}/leg_v2.stl" />
+    <xacro:property name="foot_mesh" value="${mesh_dir}/piedino_v3.STL" />
+    <xacro:property name="realsense_mesh" value="${mesh_dir}/realsense.stl" />
+    <material name="black">
+        <color rgba="0.9 0.9 0.9 1.0" />
+    </material>
+    <material name="gray">
+        <color rgba="0 0 0 0.8" />
+    </material>
+    <material name="green">
+        <color rgba="0 1 0 0.8" />
+    </material>
+    <material name="red">
+        <color rgba="1 0 0 0.8" />
+    </material>
 </robot>
